File: cpu.sch (KiCad schematic (older format))
At the start: 13 parts, among them J3 HE10-20, J4 HE10-34, Q2 DS1813, SW1 SW_Push, SW2 SW_Push, U4 WD65C02PLCC44, U5 WD65C22PLCC44

Commit message: Update to schema.
Other:
- note added: "Add a DS1813 as button debouncer"
Changed lines of the file:
@@
 EESchema Schematic File Version 4
 LIBS:OricAtmos-cache
-EELAYER 26 0
+EELAYER 29 0
 EELAYER END
 $Descr A4 11693 8268
@@
 Wire Bus Line
 	1600 900  1600 2400
+Text Notes 1200 5150 0    50   ~ 0
+Add a DS1813 as button debouncer
 $EndSCHEMATC
