File: power.sch (KiCad schematic (older format))
At the start: 5 parts, among them J1 Barrel_Jack, U1 LM7805_TO220

Commit message: Update to schema.
Other:
- note added: "Add fuse and power on switch."
Changed lines of the file:
@@
 EESchema Schematic File Version 4
 LIBS:OricAtmos-cache
-EELAYER 26 0
+EELAYER 29 0
 EELAYER END
 $Descr A4 11693 8268
@@
 $EndComp
 Wire Wire Line
-	1850 1375 3825 1375
+	1850 1375 2025 1375
 Wire Wire Line
 	1850 1275 2025 1275
@@
 	2300 1175 2300 1025
 Wire Wire Line
-	2300 1025 2625 1025
+	2300 1025 2475 1025
 $Comp
 L OricAtmos-rescue:+9V #PWR2
@@
 $EndComp
 Wire Wire Line
-	3225 1025 3800 1025
+	3225 1025 3300 1025
 $Comp
 L OricAtmos-rescue:VCC #PWR03
@@
 Text HLabel 2700 3400 2    60   Output ~ 0
 ~MAP
+Wire Wire Line
+	2025 1375 2475 1375
+Wire Wire Line
+	2925 1375 3300 1375
+Wire Wire Line
+	2475 1025 2625 1025
+Wire Wire Line
+	2475 1375 2925 1375
+Wire Wire Line
+	3300 1375 3825 1375
+Wire Wire Line
+	3300 1025 3800 1025
+Text Notes 1300 775  0    50   ~ 0
+Add fuse and power on switch.
 $EndSCHEMATC
