File: tape.sch (KiCad schematic (older format))
At the start: 0 parts

Commit message: Update to schema.
Parts:
- added C? (x2): 47nF, symbol Device:C_Small
- added C?: 100nF, symbol Device:C_Small
- added C?: C_Small, symbol Device:C_Small
- added D? (x3): DIODE, symbol Device:D_Small_ALT
- added J?: DIN-7, symbol Connector:DIN-7
- added JP?: JUMPER, symbol Jumper:Jumper_2_Open
- added JP?: Jumper_2_Open, symbol Jumper:Jumper_2_Open
- added Q? (x2): 2SC1815, symbol Device:Q_NPN_ECB
- added R? (x5): 10k, symbol Device:R_Small
- added R?: 12k, symbol Device:R_Small
- added R? (x3): 1k, symbol Device:R_Small
- added R?: 100k, symbol Device:R_Small
- added R?: 22k, symbol Device:R_Small
- added U? (x4): LM358, symbol Amplifier_Operational:LM358
Connections:
- new net: D?.1 (K), D?.2 (A), R?.1, R?.2, U?.2 (-)
- new net: C?.2, R?.2
- new net: C?.2, D?.1 (K), D?.2 (A), R?.2, R?.2, U?.3 (+), U?.6 (-)
- new net: R?.1, R?.2
- new net: R?.1, R?.2, U?.1
- new net: R?.1, R?.1, U?.5 (+)
- new net: Q?.3 (B), R?.2
- new net CB1: C?.1, Q?.2 (C), R?.2
- new net GND: C?.1, C?.2, C?.2, D?.1 (K), J?.2, Q?.1 (E), Q?.1 (E), R?.1, R?.2, U?.4 (V-), U?.4 (V-)
- new net PB6: Q?.3 (B)
- new net PB7: R?.2
- new net SOUND_OUT: J?.4, J?.5
- new net TAPE_AMP: R?.2, U?.7
- new net TAPE_IN: C?.1, J?.3
- new net TAPE_OUT: C?.1, J?.1, R?.1, R?.1
- new net VCC: R?.1, R?.1, U?.8 (V+), U?.8 (V+)
- new net relay12: J?.7
- new net relay16: J?.6
- new net relay3: JP?.2 (B)
- new net relay5: R?.1
- new net relay9: D?.2 (A), Q?.2 (C)
Other:
- note added: "Shunt jumper only you want\nto support VSYNC\n"
