File: ula.sch (KiCad schematic (older format))
At the start: 11 parts, among them U6 74HC04, U7 HSC10017, U8 74LS257, U9 74LS257, Y1 12MHz

Commit message: Update to schema.
Other:
- note added: "Phi2O and Phi1O are not connected\non the MPU and not checked by WDC"
- note removed: "Phi2O and Phi1O are not connected\nand not checked by WDC"
Changed lines of the file:
@@
 EESchema Schematic File Version 4
 LIBS:OricAtmos-cache
-EELAYER 26 0
+EELAYER 29 0
 EELAYER END
 $Descr A4 11693 8268
@@
 	9250 3425 9550 3425
 Wire Bus Line
-	9650 850  9650 3325
-Wire Bus Line
 	9650 850  10300 850
 Wire Wire Line
@@
 	2075 1950 2300 1950
 Wire Wire Line
-	3200 1550 3200 2400
+	3200 1550 3200 1950
 Wire Wire Line
 	3200 1550 2100 1550
@@
 	775  1550 1800 1550
 Wire Wire Line
-	775  1550 775  2350
+	775  1550 775  1950
 Wire Wire Line
 	775  2350 1100 2350
@@
 	3625 2975 3625 3075
 Wire Wire Line
-	3625 3075 4475 3075
+	3625 3075 3900 3075
 Wire Wire Line
 	3900 2975 3900 3075
@@
 	6000 5175 6300 5175
 Wire Bus Line
-	4075 4375 4075 5075
-Wire Bus Line
 	4075 4375 3150 4375
 Wire Bus Line
-	4075 3375 4075 4075
-Wire Bus Line
 	4075 3375 3150 3375
 Wire Wire Line
 	7750 2075 7575 2075
 Wire Wire Line
-	7575 2075 7575 3975
+	7575 2075 7575 3625
 Wire Wire Line
 	7750 3625 7575 3625
@@
 	7750 2175 7675 2175
 Wire Wire Line
-	7675 2175 7675 3925
+	7675 2175 7675 3725
 Wire Wire Line
 	7750 3725 7675 3725
@@
 	7200 3375 7750 3375
 Wire Bus Line
-	6400 2975 6400 3675
-Wire Bus Line
 	6400 3675 7100 3675
-Wire Bus Line
-	7100 3675 7100 975
 Wire Wire Line
 	7750 1175 6900 1175
@@
 Entry Wire Line
 	6800 3375 6900 3475
-Wire Bus Line
-	6800 3375 6800 975
 Wire Bus Line
 	6800 975  6200 975
@@
 Phi2
 Text Notes 4050 2475 0    60   ~ 12
-Phi2O and Phi1O are not connected\nand not checked by WDC
+Phi2O and Phi1O are not connected\non the MPU and not checked by WDC
 $Comp
 L OricAtmos-rescue:C_Small C12
@@
 Text HLabel 4175 4325 0    60   Input ~ 0
 R/~W
+Wire Wire Line
+	775  1950 775  2350
+Wire Wire Line
+	3200 1950 3200 2400
+Wire Wire Line
+	3900 3075 4475 3075
+Wire Wire Line
+	7575 3625 7575 3975
+Wire Wire Line
+	7675 3725 7675 3925
+Wire Bus Line
+	4075 3375 4075 4075
+Wire Bus Line
+	4075 4375 4075 5075
+Wire Bus Line
+	6400 2975 6400 3675
+Wire Bus Line
+	9650 850  9650 3325
+Wire Bus Line
+	7100 975  7100 3675
+Wire Bus Line
+	6800 975  6800 3375
 $EndSCHEMATC
