File: OricAtmos.sch (KiCad schematic (older format))
At the start: 0 parts

Commit message: added OSDK and cumulus projects
Changed lines of the file:
@@
 F0 "Tape" 60
 F1 "tape.sch" 60
+F2 "PB[0..7]" I R 2675 3950 50
+F3 "SYNC_IN" I R 2675 4300 50
+F4 "CB1" O R 2675 4100 50
+F5 "SOUND_OUT" I L 1175 4000 50
 $EndSheet
 $Sheet
@@
 	2650 2950 3400 2950
 Wire Bus Line
-	2650 3200 3400 3200
+	2650 3200 2775 3200
 Text Label 2800 2825 0    60   ~ 0
 CA2
@@
 Wire Wire Line
 	5525 2950 5900 2950
+Wire Bus Line
+	2775 3200 2775 3950
+Wire Bus Line
+	2775 3950 2675 3950
+Connection ~ 2775 3200
+Wire Bus Line
+	2775 3200 3400 3200
+Wire Wire Line
+	3400 3325 2850 3325
+Wire Wire Line
+	2850 3325 2850 4100
+Wire Wire Line
+	2850 4100 2675 4100
+Wire Wire Line
+	10300 2525 10850 2525
+Wire Wire Line
+	10850 2525 10850 4500
+Wire Wire Line
+	10850 4500 2850 4500
+Wire Wire Line
+	2850 4500 2850 4300
+Wire Wire Line
+	2850 4300 2675 4300
+Wire Wire Line
+	1175 4000 875  4000
+Wire Wire Line
+	875  4000 875  2950
+Connection ~ 875  2950
 $EndSCHEMATC
